Commit message: robot core update

File: description/robot_core.xacro (robot description, xacro)
@@ -2,11 +2,4 @@
 <robot xmlns:xacro="http://www.ros.org/wiki/xacro" >
     <xacro:include filename="inertial_macros.xacro"/>
-    <xacro:property name="rover_length" value="0.302"/>
-    <xacro:property name="rover_width" value="0.201"/>
-    <xacro:property name="rover_height" value="0.054"/>
-    <xacro:property name="rover_mass" value="1.0"/>
-    <xacro:property name="wheel_radius" value="0.036"/>
-    <xacro:property name="wheel_thickness" value="0.037"/>
-    <xacro:property name="wheel_mass" value="0.05"/>
     <material name="white">
         <color rgba="1.0 1.0 1.0 1.0"/>
@@ -39,5 +32,5 @@
             <origin xyz="0.0 0.0 0.01" rpy="0.0 0.0 0.0"/>
             <geometry>
-                <box size="${rover_length} ${rover_width} ${rover_height}"/>
+                <box size=".3 0.2 0.035"/>
             </geometry>
             <material name="Gray">
@@ -48,8 +41,8 @@
             <origin xyz="0.0 0.0 0.0" rpy="0.0 0.0 0.0"/>
             <geometry>
-                <box size="${rover_length} ${rover_width} ${rover_height}"/>
-            </geometry>
-        </collision>
-        <xacro:inertial_box mass = "0.5"  x = "${rover_length}" y = "${rover_width}" z = "${rover_height}">
+                <box size="0.3 0.2 0.035"/>
+            </geometry>
+        </collision>
+        <xacro:inertial_box mass = "0.5"  x = "0.3" y = "0.2" z = "0.035">
             <origin xyz="0.0 0.0 0.01" rpy="0.0 0.0 0.0"/>
         </xacro:inertial_box>
@@ -97,5 +90,5 @@
         <parent link="base_link"/>
         <child link="front_left_wheel"/>
-        <origin xyz="0.075 0.119 0.0" rpy="-1.57 0.0 0.0"/>
+        <origin xyz="0.08 0.118 0.01" rpy="1.57 0.0 0.0"/>
         <axis xyz="0.0 0.0 -0.1"/>
     </joint>
@@ -103,16 +96,16 @@
         <visual>
             <geometry>
-                <cylinder radius="${wheel_radius}" length="${wheel_thickness}"/>
-            </geometry>
-            <material name="orange">
-                <color rgba="0.0 0.0 0.0 1.0"/>
-            </material>
-        </visual>
-        <collision>
-            <geometry>
-                 <cylinder radius="${wheel_radius}" length="${wheel_thickness}"/>
-            </geometry>
-        </collision>
-        <xacro:inertial_cylinder mass="${wheel_mass}" radius="${wheel_radius}" length="${wheel_thickness}">
+                <cylinder radius=".035" length="0.035"/>
+            </geometry>
+            <material name="orange">
+                <color rgba="0.0 0.0 0.0 1.0"/>
+            </material>
+        </visual>
+        <collision>
+            <geometry>
+                <cylinder radius="0.035" length="0.035"/>
+            </geometry>
+        </collision>
+        <xacro:inertial_cylinder mass="0.1" radius="0.035" length="0.035">
             <origin xyz="0.0 0.0 0.0" rpy="0.0 0.0 0.0"/>
         </xacro:inertial_cylinder>
@@ -127,5 +120,5 @@
         <parent link="base_link"/>
         <child link="front_right_wheel"/>
-        <origin xyz="0.075 -0.119 0.0" rpy="1.57 0.0 0.0"/>
+        <origin xyz="0.08 -0.118 0.01" rpy="1.57 0.0 0.0"/>
         <axis xyz="0.0 0.0 -0.1"/>
     </joint>
@@ -133,16 +126,16 @@
         <visual>
             <geometry>
-                 <cylinder radius="${wheel_radius}" length="${wheel_thickness}"/>
-            </geometry>
-            <material name="orange">
-                <color rgba="0.0 0.0 0.0 1.0"/>
-            </material>
-        </visual>
-        <collision>
-            <geometry>
-                <cylinder radius="${wheel_radius}" length="${wheel_thickness}"/>
-            </geometry>
-        </collision>
-        <xacro:inertial_cylinder mass="${wheel_mass}" radius="${wheel_radius}" length="${wheel_thickness}">
+                <cylinder radius=".035" length="0.035"/>
+            </geometry>
+            <material name="orange">
+                <color rgba="0.0 0.0 0.0 1.0"/>
+            </material>
+        </visual>
+        <collision>
+            <geometry>
+                <cylinder radius="0.035" length="0.035"/>
+            </geometry>
+        </collision>
+        <xacro:inertial_cylinder mass="0.1" radius="0.035" length="0.035">
             <origin xyz="0.0 0.0 0.0" rpy="0.0 0.0 0.0"/>
         </xacro:inertial_cylinder>
@@ -157,5 +150,5 @@
         <parent link="base_link"/>
         <child link="back_left_wheel"/>
-        <origin xyz="-0.075 0.119 0.0" rpy="-1.57 0.0 0.0"/>
+        <origin xyz="-0.08 0.118 0.01" rpy="1.57 0.0 0.0"/>
         <axis xyz="0.0 0.0 -0.1"/>
     </joint>
@@ -163,16 +156,16 @@
         <visual>
             <geometry>
-                <cylinder radius="${wheel_radius}" length="${wheel_thickness}"/>
-            </geometry>
-            <material name="orange">
-                <color rgba="0.0 0.0 0.0 1.0"/>
-            </material>
-        </visual>
-        <collision>
-            <geometry>
-                <cylinder radius="${wheel_radius}" length="${wheel_thickness}"/>
-            </geometry>
-        </collision>
-        <xacro:inertial_cylinder mass="${wheel_mass}" radius="${wheel_radius}" length="${wheel_thickness}">
+                <cylinder radius=".035" length="0.035"/>
+            </geometry>
+            <material name="orange">
+                <color rgba="0.0 0.0 0.0 1.0"/>
+            </material>
+        </visual>
+        <collision>
+            <geometry>
+                <cylinder radius="0.035" length="0.035"/>
+            </geometry>
+        </collision>
+        <xacro:inertial_cylinder mass="0.1" radius="0.035" length="0.035">
             <origin xyz="0.0 0.0 0.0" rpy="0.0 0.0 0.0"/>
         </xacro:inertial_cylinder>
@@ -187,5 +180,5 @@
         <parent link="base_link"/>
         <child link="back_right_wheel"/>
-        <origin xyz="-0.075 -0.119 0.0" rpy="1.57 0.0 0.0"/>
+        <origin xyz="-0.08 -0.118 0.01" rpy="1.57 0.0 0.0"/>
         <axis xyz="0.0 0.0 -0.1"/>
     </joint>
@@ -193,16 +186,16 @@
         <visual>
             <geometry>
-                <cylinder radius="${wheel_radius}" length="${wheel_thickness}"/>
-            </geometry>
-            <material name="orange">
-                <color rgba="0.0 0.0 0.0 1.0"/>
-            </material>
-        </visual>
-        <collision>
-            <geometry>
-                <cylinder radius="${wheel_radius}" length="${wheel_thickness}"/>
-            </geometry>
-        </collision>
-        <xacro:inertial_cylinder mass="${wheel_mass}" radius="${wheel_radius}" length="${wheel_thickness}">
+                <cylinder radius=".035" length="0.035"/>
+            </geometry>
+            <material name="orange">
+                <color rgba="0.0 0.0 0.0 1.0"/>
+            </material>
+        </visual>
+        <collision>
+            <geometry>
+                <cylinder radius="0.035" length="0.035"/>
+            </geometry>
+        </collision>
+        <xacro:inertial_cylinder mass="0.1" radius="0.035" length="0.035">
             <origin xyz="0.0 0.0 0.0" rpy="0.0 0.0 0.0"/>
         </xacro:inertial_cylinder>
