Commit message: wheel control

File: description/robot.urdf.xacro (robot description, xacro)
@@ -1,4 +1,6 @@
 <?xml version="1.0"?>
-<robot xmlns:xacro="http://www.ros.org/wiki/xacro"  name="robot">
+<robot xmlns:xacro="http://www.ros.org/wiki/xacro"  name="rover">
     <xacro:include filename="rover_core.xacro"/>
+    <xacro:include filename="front_wheel_gazebo_control.xacro"/>
+    <xacro:include filename="back_wheel_gazebo_control.xacro"/>
 </robot>

File: description/rover_core.xacro (robot description, xacro)
@@ -1,4 +1,4 @@
 <?xml version="1.0"?>
-<robot xmlns:xacro="http://www.ros.org/wiki/xacro" name="robot_name">
+<robot xmlns:xacro="http://www.ros.org/wiki/xacro" >
     <xacro:include filename="inertial_macros.xacro"/>
     <material name="white">
@@ -14,6 +14,12 @@
         <color rgba="0.0 0.0 0.0 1.0"/>
     </material>
+    <material name="Gray">
+        <color rgba="0.3 0.3 0.3 1.0"/>
+    </material>
     <!-- Base Link -->
     <link name="base_link">
+        <visual>
+            <origin xyz="0.0 0.0 0.0" rpy="0.0 0.0 0.0"/>
+        </visual>
     </link>
     <joint name="chassis_joint" type="fixed">
@@ -31,14 +37,28 @@
                 <box size=".3 0.2 0.035"/>
             </geometry>
-            <material name="white">
-                <color rgba="0.0 0.0 0.0 1.0"/>
+            <material name="Gray">
+                <color rgba="0.3 0.3 0.3 1.0"/>
             </material>
         </visual>
+        <collision>
+            <origin xyz="0.0 0.0 0.0" rpy="0.0 0.0 0.0"/>
+            <geometry>
+                <box size="0.3 0.2 0.035"/>
+            </geometry>
+        </collision>
+        <xacro:inertial_box mass = "0.5"  x = "0.3" y = "0.2" z = "0.035">
+            <origin xyz="0.0 0.0 0.01" rpy="0.0 0.0 0.0"/>
+        </xacro:inertial_box>
     </link>
+    <gazebo reference = "chassis">
+        <material>
+            Gazebo/Gray
+        </material>
+    </gazebo>
     <!--  Front Left Wheel Link-->
     <joint name="front_left_wheel_joint" type="continuous">
         <parent link="base_link"/>
         <child link="front_left_wheel"/>
-        <origin xyz="0.1 0.118 0" rpy="-1.57 0.0 0.0"/>
+        <origin xyz="0.08 0.118 0.01" rpy="-1.57 0.0 0.0"/>
         <axis xyz="0.0 0.0 -0.1"/>
     </joint>
@@ -49,12 +69,26 @@
             </geometry>
             <material name="orange">
+                <color rgba="0.0 0.0 0.0 1.0"/>
             </material>
         </visual>
+        <collision>
+            <geometry>
+                <cylinder radius="0.035" length="0.035"/>
+            </geometry>
+        </collision>
+        <xacro:inertial_cylinder mass="0.1" radius="0.035" length="0.035">
+            <origin xyz="0.0 0.0 0.0" rpy="0.0 0.0 0.0"/>
+        </xacro:inertial_cylinder>
     </link>
+    <gazebo reference = "front_left_wheel">
+        <material>
+            Gazebo/Orange
+        </material>
+    </gazebo>
     <!-- Front Right Wheel Link -->
     <joint name="front_right_wheel_joint" type="continuous">
         <parent link="base_link"/>
         <child link="front_right_wheel"/>
-        <origin xyz="0.1 -0.118 0.0" rpy="-1.57 0.0 0.0"/>
+        <origin xyz="0.08 -0.118 0.01" rpy="1.57 0.0 0.0"/>
         <axis xyz="0.0 0.0 -0.1"/>
     </joint>
@@ -68,10 +102,23 @@
             </material>
         </visual>
+        <collision>
+            <geometry>
+                <cylinder radius="0.035" length="0.035"/>
+            </geometry>
+        </collision>
+        <xacro:inertial_cylinder mass="0.1" radius="0.035" length="0.035">
+            <origin xyz="0.0 0.0 0.0" rpy="0.0 0.0 0.0"/>
+        </xacro:inertial_cylinder>
     </link>
+    <gazebo reference = "front_right_wheel">
+        <material>
+            Gazebo/Orange
+        </material>
+    </gazebo>
     <!-- Back Left Wheel Link  -->
     <joint name="back_left_wheel_joint" type="continuous">
         <parent link="base_link"/>
         <child link="back_left_wheel"/>
-        <origin xyz="-0.1 0.118 0.0" rpy="-1.57 0.0 0.0"/>
+        <origin xyz="-0.08 0.118 0.01" rpy="-1.57 0.0 0.0"/>
         <axis xyz="0.0 0.0 -0.1"/>
     </joint>
@@ -85,10 +132,23 @@
             </material>
         </visual>
+        <collision>
+            <geometry>
+                <cylinder radius="0.035" length="0.035"/>
+            </geometry>
+        </collision>
+        <xacro:inertial_cylinder mass="0.1" radius="0.035" length="0.035">
+            <origin xyz="0.0 0.0 0.0" rpy="0.0 0.0 0.0"/>
+        </xacro:inertial_cylinder>
     </link>
+    <gazebo reference = "back_left_wheel">
+        <material>
+            Gazebo/Orange
+        </material>
+    </gazebo>
     <!-- Back Right Wheel Link -->
     <joint name="back_right_wheel_joint" type="continuous">
         <parent link="base_link"/>
         <child link="back_right_wheel"/>
-        <origin xyz="-0.1 -0.118 0.0" rpy="-1.57 0.0 0.0"/>
+        <origin xyz="-0.08 -0.118 0.01" rpy="1.57 0.0 0.0"/>
         <axis xyz="0.0 0.0 -0.1"/>
     </joint>
@@ -102,4 +162,17 @@
             </material>
         </visual>
+        <collision>
+            <geometry>
+                <cylinder radius="0.035" length="0.035"/>
+            </geometry>
+        </collision>
+        <xacro:inertial_cylinder mass="0.1" radius="0.035" length="0.035">
+            <origin xyz="0.0 0.0 0.0" rpy="0.0 0.0 0.0"/>
+        </xacro:inertial_cylinder>
     </link>
+    <gazebo reference = "back_right_wheel">
+        <material>
+            Gazebo/Orange
+        </material>
+    </gazebo>
     </robot>

Commit message: update

File: description/robot.urdf.xacro (robot description, xacro)
@@ -2,4 +2,5 @@
 <robot xmlns:xacro="http://www.ros.org/wiki/xacro"  name="rover">
     <xacro:include filename="rover_core.xacro"/>
+    <!-- <xacro:include filename="robot_core.xacro"/> -->
     <!-- <xacro:include filename="wheel_gazebo_control.xacro"/> -->
     <!-- <xacro:include filename="back_wheel_gazebo_control.xacro"/> -->

File: description/rover_core.xacro (robot description, xacro)
@@ -8,5 +8,5 @@
     <xacro:property name="wheel_radius" value="0.036"/>
     <xacro:property name="wheel_thickness" value="0.037"/>
-    <xacro:property name="wheel_mass" value="0.05"/>
+    <xacro:property name="wheel_mass" value="0.04"/>
     <material name="white">
         <color rgba="1.0 1.0 1.0 1.0"/>
@@ -37,5 +37,5 @@
     <link name="chassis">
         <visual>
-            <origin xyz="0.0 0.0 0.01" rpy="0.0 0.0 0.0"/>
+            <origin xyz="0.0 0.0 ${rover_height/2}" rpy="0.0 0.0 0.0"/>
             <geometry>
                 <box size="${rover_length} ${rover_width} ${rover_height}"/>
@@ -46,5 +46,5 @@
         </visual>
         <collision>
-            <origin xyz="0.0 0.0 0.0" rpy="0.0 0.0 0.0"/>
+            <origin xyz="0.0 0.0 0.01" rpy="0.0 0.0 0.0"/>
             <geometry>
                 <box size="${rover_length} ${rover_width} ${rover_height}"/>
@@ -52,5 +52,5 @@
         </collision>
         <xacro:inertial_box mass = "0.5"  x = "${rover_length}" y = "${rover_width}" z = "${rover_height}">
-            <origin xyz="0.0 0.0 0.01" rpy="0.0 0.0 0.0"/>
+            <origin xyz="0.0 0.0 ${rover_height/2}" rpy="0.0 0.0 0.0"/>
         </xacro:inertial_box>
     </link>
@@ -74,17 +74,8 @@
                 <box size=".02 0.02 0.02"/>
             </geometry>
-            <material name="Gray">
+            <material name="blue">
                 <color rgba="0.3 0.3 0.3 1.0"/>
             </material>
         </visual>
-        <collision>
-            <origin xyz="0.0 0.0 0.0" rpy="0.0 0.0 0.0"/>
-            <geometry>
-                <box size="0.3 0.2 0.035"/>
-            </geometry>
-        </collision>
-        <xacro:inertial_box mass = "0.5"  x = "0.3" y = "0.2" z = "0.035">
-            <origin xyz="0.0 0.0 0.01" rpy="0.0 0.0 0.0"/>
-        </xacro:inertial_box>
     </link>
     <gazebo reference = "Front">
@@ -97,5 +88,5 @@
         <parent link="base_link"/>
         <child link="front_left_wheel"/>
-        <origin xyz="0.075 0.119 0.0" rpy="-1.57 0.0 0.0"/>
+        <origin xyz="0.075 0.140 0.0" rpy="1.57 0.0 0.0"/>
         <axis xyz="0.0 0.0 -0.1"/>
     </joint>
@@ -111,5 +102,5 @@
         <collision>
             <geometry>
-                 <cylinder radius="${wheel_radius}" length="${wheel_thickness}"/>
+                <sphere  radius="${wheel_radius}"/>
             </geometry>
         </collision>
@@ -127,5 +118,5 @@
         <parent link="base_link"/>
         <child link="front_right_wheel"/>
-        <origin xyz="0.075 -0.119 0.0" rpy="1.57 0.0 0.0"/>
+        <origin xyz="0.075 -0.140 0.0" rpy="1.57 0.0 0.0"/>
         <axis xyz="0.0 0.0 -0.1"/>
     </joint>
@@ -133,13 +124,13 @@
         <visual>
             <geometry>
-                 <cylinder radius="${wheel_radius}" length="${wheel_thickness}"/>
-            </geometry>
-            <material name="orange">
-                <color rgba="0.0 0.0 0.0 1.0"/>
-            </material>
-        </visual>
-        <collision>
-            <geometry>
-                <cylinder radius="${wheel_radius}" length="${wheel_thickness}"/>
+                <cylinder radius="${wheel_radius}" length="${wheel_thickness}"/>
+            </geometry>
+            <material name="orange">
+                <color rgba="0.0 0.0 0.0 1.0"/>
+            </material>
+        </visual>
+        <collision>
+            <geometry>
+                <sphere  radius="${wheel_radius}" />
             </geometry>
         </collision>
@@ -157,5 +148,5 @@
         <parent link="base_link"/>
         <child link="back_left_wheel"/>
-        <origin xyz="-0.075 0.119 0.0" rpy="-1.57 0.0 0.0"/>
+        <origin xyz="-0.075 0.140 0.0" rpy="1.57 0.0 0.0"/>
         <axis xyz="0.0 0.0 -0.1"/>
     </joint>
@@ -171,5 +162,5 @@
         <collision>
             <geometry>
-                <cylinder radius="${wheel_radius}" length="${wheel_thickness}"/>
+                <sphere  radius="${wheel_radius}"/>
             </geometry>
         </collision>
@@ -187,5 +178,5 @@
         <parent link="base_link"/>
         <child link="back_right_wheel"/>
-        <origin xyz="-0.075 -0.119 0.0" rpy="1.57 0.0 0.0"/>
+        <origin xyz="-0.075 -0.140 0.0" rpy="1.57 0.0 0.0"/>
         <axis xyz="0.0 0.0 -0.1"/>
     </joint>
@@ -201,5 +192,5 @@
         <collision>
             <geometry>
-                <cylinder radius="${wheel_radius}" length="${wheel_thickness}"/>
+                <sphere  radius="${wheel_radius}"/>
             </geometry>
         </collision>

Commit message: real rover control

File: description/robot.urdf.xacro (robot description, xacro)
@@ -5,4 +5,4 @@
     <!-- <xacro:include filename="wheel_gazebo_control.xacro"/> -->
     <!-- <xacro:include filename="back_wheel_gazebo_control.xacro"/> -->
-    <xacro:include filename="ros2_control.xacro"/>
+    <xacro:include filename="ros2_real_bot_control.xacro"/>
 </robot>

File: description/ros2_control.xacro (robot description, xacro)
@@ -1,5 +1,5 @@
 <?xml version="1.0"?>
 <robot xmlns:xacro="http://www.ros.org/wiki/xacro">
-    <ros2_control name="RealRobot" type="system">
+    <!-- <ros2_control name="RealRobot" type="system">
         <hardware>
             <plugin>diffdrive_arduino/DiffDriveArduino</plugin>
@@ -13,7 +13,7 @@
             <param name="timeout">1000</param>
             <param name="enc_counts_per_rev">3436</param>
-        </hardware>
+        </hardware> -->
         <!-- Note everything below here is the same as the Gazebo one -->
-        <joint name="front_left_wheel_joint">
+        <!-- <joint name="front_left_wheel_joint">
             <command_interface name="velocity">
                 <param name="min">-10</param>
@@ -47,6 +47,6 @@
             <state_interface name="position" />
         </joint>
-    </ros2_control>
-    <!-- <ros2_control name="GazeboSystem" type="system">
+    </ros2_control> -->
+    <ros2_control name="GazeboSystem" type="system">
         <hardware>
             <plugin>gazebo_ros2_control/GazeboSystem</plugin>
@@ -84,5 +84,5 @@
             <state_interface name="position" />
         </joint>
-``  </ros2_control> -->
+``  </ros2_control>
     <gazebo>
         <plugin filename="libgazebo_ros2_control.so" name="gazebo_ros2_control">

File: description/rover_core.xacro (robot description, xacro)
@@ -61,5 +61,5 @@
     </gazebo>
     <!-- front face Link -->
-    <joint name="front_face_joint" type="fixed">
+    <joint name="face_joint" type="fixed">
         <origin xyz="0.0 0.0 0.0" rpy="0.0 0.0 0.0"/>
         <parent link="base_link"/>
@@ -85,11 +85,11 @@
     </gazebo>
     <!--  Front Left Wheel Link-->
-    <joint name="front_left_wheel_joint" type="continuous">
-        <parent link="base_link"/>
-        <child link="front_left_wheel"/>
+    <joint name="left_wheel_joint" type="continuous">
+        <parent link="base_link"/>
+        <child link="left_wheel"/>
         <origin xyz="0.075 0.140 0.0" rpy="1.57 0.0 0.0"/>
         <axis xyz="0.0 0.0 -0.1"/>
     </joint>
-    <link name="front_left_wheel">
+    <link name="left_wheel">
         <visual>
             <geometry>
@@ -109,5 +109,5 @@
         </xacro:inertial_cylinder>
     </link>
-    <gazebo reference = "front_left_wheel">
+    <gazebo reference = "left_wheel">
         <material>
             Gazebo/Orange
@@ -115,11 +115,11 @@
     </gazebo>
     <!-- Front Right Wheel Link -->
-    <joint name="front_right_wheel_joint" type="continuous">
-        <parent link="base_link"/>
-        <child link="front_right_wheel"/>
+    <joint name="right_wheel_joint" type="continuous">
+        <parent link="base_link"/>
+        <child link="right_wheel"/>
         <origin xyz="0.075 -0.140 0.0" rpy="1.57 0.0 0.0"/>
         <axis xyz="0.0 0.0 -0.1"/>
     </joint>
-    <link name="front_right_wheel">
+    <link name="right_wheel">
         <visual>
             <geometry>
@@ -139,5 +139,5 @@
         </xacro:inertial_cylinder>
     </link>
-    <gazebo reference = "front_right_wheel">
+    <gazebo reference = "right_wheel">
         <material>
             Gazebo/Orange
@@ -145,5 +145,5 @@
     </gazebo>
     <!-- Back Left Wheel Link  -->
-    <joint name="back_left_wheel_joint" type="continuous">
+    <!-- <joint name="back_left_wheel_joint" type="continuous">
         <parent link="base_link"/>
         <child link="back_left_wheel"/>
@@ -173,7 +173,7 @@
             Gazebo/Orange
         </material>
-    </gazebo>
+    </gazebo> -->
     <!-- Back Right Wheel Link -->
-    <joint name="back_right_wheel_joint" type="continuous">
+    <!-- <joint name="back_right_wheel_joint" type="continuous">
         <parent link="base_link"/>
         <child link="back_right_wheel"/>
@@ -203,4 +203,4 @@
             Gazebo/Orange
         </material>
-    </gazebo>
+    </gazebo> -->
     </robot>
